File: DualUSBHub/DualUSBHub.kicad_pcb (KiCad board)
At the start: 2 copper layers, 44 parts, among them J1 USB_A, J2 USB_A, J3 USB_A, J4 USB_A, J5 USB_OTG, J6 USB_OTG, SW1 SW_DIP_x01, SW2 SW_DIP_x01, U1 CH440G, U2 CH440G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

Commit message: update; add a dual switch
Parts:
- moved D1 91.7 mm to (105.4, 57.1)
- moved R1 78.7 mm to (86.4, 146.1), turned to 270 degrees
- moved R8 72.6 mm to (100.3, 57.1), turned to 180 degrees
- moved D2 71.1 mm to (105.4, 53.3), turned to 180 degrees
- moved C7 70.4 mm to (90.2, 71.1)
- moved R5 69.1 mm to (90.2, 73.7)
- moved D4 63.6 mm to (149.9, 48.3), turned to 180 degrees
- moved R7 59.1 mm to (144.8, 52.1), turned to 180 degrees
- moved C10 56.9 mm to (163.8, 72.4)
- moved D3 56.4 mm to (149.9, 52.1)
- moved D5 56.1 mm to (132.1, 58.4)
- moved R2 52.3 mm to (130.8, 146.1), turned to 270 degrees
- moved R10 46.3 mm to (126.7, 66.0), turned to 180 degrees
- moved Y1 46.2 mm to (52.1, 92.7), turned to 180 degrees
- moved R11 45.9 mm to (161.3, 61.0)
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Routing:
- net GND: track 0.00 -> 165.2 mm
- net Net-(U4-Pad2): track 0.00 -> 101.5 mm
- net Net-(U4-Pad3): track 0.00 -> 94.3 mm
- net VBUS: track 0.00 -> 46.4 mm
- net Net-(U3-Pad2): track 0.00 -> 33.5 mm
- net Net-(U3-Pad3): track 0.00 -> 25.5 mm
- net VCC: track 0.00 -> 14.3 mm
- net SRSTA: track 0.00 -> 13.9 mm
- net Net-(R2-Pad1): track 0.00 -> 11.5 mm
- net DRVB: track 0.00 -> 11.4 mm
- net Net-(D5-Pad1): track 0.00 -> 11.0 mm
- net Net-(R1-Pad1): track 0.00 -> 9.94 mm
- net Net-(D7-Pad1): track 0.00 -> 8.11 mm
- net DRVA: track 0.00 -> 7.62 mm
- net Net-(D3-Pad1): track 0.00 -> 6.84 mm
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