File: DualUSBHub/DualUSBHub.sch (KiCad schematic (older format))
At the start: 26 parts, among them J1 USB_A, J2 USB_A, J3 USB_A, J4 USB_A, J5 USB_OTG, J6 USB_OTG, SW1 SW_DIP_x01, SW2 SW_DIP_x01, U1 CH440G, U2 CH440G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

Commit message: update; add a dual switch
Parts:
- U1, U2: footprint DualUSBHub:ch440g -> lib:ch440g
- U3, U4: footprint DualUSBHub:ma8601 -> lib:ma8601
Changed lines of the file:
@@
 EESchema Schematic File Version 2
+LIBS:ch440g
+LIBS:ma8601
 LIBS:power
 LIBS:device
@@
 LIBS:contrib
 LIBS:valves
-LIBS:ma8601
-LIBS:ch440g
 LIBS:DualUSBHub-cache
 EELAYER 25 0
@@
 F 0 "U3" H 5700 2250 60  0000 C CNN
 F 1 "MA8601" H 5700 750 60  0000 C CNN
-F 2 "DualUSBHub:ma8601" H 5700 1700 60  0001 C CNN
+F 2 "lib:ma8601" H 5700 1700 60  0001 C CNN
 F 3 "" H 5700 1700 60  0001 C CNN
 	1    5700 1500
@@
 F 0 "U2" H 2850 4950 60  0000 C CNN
 F 1 "CH440G" H 2850 4050 60  0000 C CNN
-F 2 "DualUSBHub:ch440g" H 2850 4550 60  0001 C CNN
+F 2 "lib:ch440g" H 2850 4550 60  0001 C CNN
 F 3 "" H 2850 4550 60  0001 C CNN
 	1    2850 4550
@@
 F 0 "U1" H 2800 3700 60  0000 C CNN
 F 1 "CH440G" H 2800 2800 60  0000 C CNN
-F 2 "DualUSBHub:ch440g" H 2800 3300 60  0001 C CNN
+F 2 "lib:ch440g" H 2800 3300 60  0001 C CNN
 F 3 "" H 2800 3300 60  0001 C CNN
 	1    2800 3300
@@
 F 0 "U4" H 5700 5350 60  0000 C CNN
 F 1 "MA8601" H 5700 3850 60  0000 C CNN
-F 2 "DualUSBHub:ma8601" H 5700 4800 60  0001 C CNN
+F 2 "lib:ma8601" H 5700 4800 60  0001 C CNN
 F 3 "" H 5700 4800 60  0001 C CNN
 	1    5700 4600
