File: QuadUSBSwitch/QuadUSBSwitch.kicad_pcb (KiCad board)
At the start: 2 copper layers, 15 parts, among them J1 USB_A, J2 USB_A, J3 USB_OTG, J4 USB_OTG, J5 USB_OTG, J6 USB_OTG, J7 USB_OTG, SW1 SW_DIP_x04, U1 CH440G

Commit message: update;
Parts:
- moved J3 1.71 mm to (115.8, 63.8), turned to 180 degrees
Routing:
- net Net-(J3-Pad6): track 11.4 -> 13.4 mm
- net VBUS: track 80.8 -> 79.9 mm
- net GND: track 162.1 -> 162.7 mm
Changed lines of the file:
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@@
 (kicad_pcb (version 4) (host pcbnew 4.0.7)
   (general
-    (links 0)
+    (links 59)
     (no_connects 0)
-    (area 70.984999 57.985 133.135 104.675)
+    (area 70.984999 56.215 133.135 103.275)
     (thickness 1.6)
     (drawings 0)
-    (tracks 205)
+    (tracks 207)
     (zones 0)
     (modules 15)
@@
   )
   (module Connectors:USB_Micro-B (layer F.Cu)
-    (at 116.4 62.2)
+    (at 115.8 63.8 180)
     (descr "Micro USB Type B Receptacle")
     (tags "USB USB_B USB_micro USB_OTG")
     (attr smd)
-    (fp_text reference J3 (at 0 -3.24) (layer F.SilkS)
-      (effects (font (size 1 1) (thickness 0.15)))
-    )
-    (fp_text value USB_OTG (at 0 5.01) (layer F.Fab)
+    (fp_text reference J3 (at 0 -3.24 180) (layer F.SilkS)
+      (effects (font (size 1 1) (thickness 0.15)))
+    )
+    (fp_text value USB_OTG (at 0 5.01 180) (layer F.Fab)
       (effects (font (size 1 1) (thickness 0.15)))
     )
@@
     (fp_line (start 4.35 2.8) (end -4.35 2.8) (layer F.SilkS) (width 0.12))
     (fp_line (start -4.35 4.03) (end -4.35 -2.38) (layer F.SilkS) (width 0.12))
-    (pad 1 smd rect (at -1.3 -1.35 90) (size 1.35 0.4) (layers F.Cu F.Paste F.Mask)
+    (pad 1 smd rect (at -1.3 -1.35 270) (size 1.35 0.4) (layers F.Cu F.Paste F.Mask)
       (net 5 VBUS))
-    (pad 2 smd rect (at -0.65 -1.35 90) (size 1.35 0.4) (layers F.Cu F.Paste F.Mask)
+    (pad 2 smd rect (at -0.65 -1.35 270) (size 1.35 0.4) (layers F.Cu F.Paste F.Mask)
       (net 6 "Net-(J3-Pad2)"))
-    (pad 3 smd rect (at 0 -1.35 90) (size 1.35 0.4) (layers F.Cu F.Paste F.Mask)
+    (pad 3 smd rect (at 0 -1.35 270) (size 1.35 0.4) (layers F.Cu F.Paste F.Mask)
       (net 7 "Net-(J3-Pad3)"))
-    (pad 4 smd rect (at 0.65 -1.35 90) (size 1.35 0.4) (layers F.Cu F.Paste F.Mask)
+    (pad 4 smd rect (at 0.65 -1.35 270) (size 1.35 0.4) (layers F.Cu F.Paste F.Mask)
       (net 8 "Net-(J3-Pad4)"))
-    (pad 5 smd rect (at 1.3 -1.35 90) (size 1.35 0.4) (layers F.Cu F.Paste F.Mask)
-      (net 9 GND))
-    (pad 6 thru_hole oval (at -2.5 -1.35 90) (size 0.95 1.25) (drill oval 0.55 0.85) (layers *.Cu *.Mask)
+    (pad 5 smd rect (at 1.3 -1.35 270) (size 1.35 0.4) (layers F.Cu F.Paste F.Mask)
+      (net 9 GND))
+    (pad 6 thru_hole oval (at -2.5 -1.35 270) (size 0.95 1.25) (drill oval 0.55 0.85) (layers *.Cu *.Mask)
       (net 10 "Net-(J3-Pad6)"))
-    (pad 6 thru_hole oval (at 2.5 -1.35 90) (size 0.95 1.25) (drill oval 0.55 0.85) (layers *.Cu *.Mask)
+    (pad 6 thru_hole oval (at 2.5 -1.35 270) (size 0.95 1.25) (drill oval 0.55 0.85) (layers *.Cu *.Mask)
       (net 10 "Net-(J3-Pad6)"))
-    (pad 6 thru_hole oval (at -3.5 1.35 90) (size 1.55 1) (drill oval 1.15 0.5) (layers *.Cu *.Mask)
+    (pad 6 thru_hole oval (at -3.5 1.35 270) (size 1.55 1) (drill oval 1.15 0.5) (layers *.Cu *.Mask)
       (net 10 "Net-(J3-Pad6)"))
-    (pad 6 thru_hole oval (at 3.5 1.35 90) (size 1.55 1) (drill oval 1.15 0.5) (layers *.Cu *.Mask)
+    (pad 6 thru_hole oval (at 3.5 1.35 270) (size 1.55 1) (drill oval 1.15 0.5) (layers *.Cu *.Mask)
       (net 10 "Net-(J3-Pad6)"))
   )
@@
   (segment (start 114.3 86.24) (end 114.299999 84.839999) (width 0.3) (layer F.Cu) (net 4))
   (via (at 115 82.2) (size 2) (drill 1) (layers F.Cu B.Cu) (net 4))
+  (segment (start 117.1 65.15) (end 117.1 66.125) (width 0.3) (layer F.Cu) (net 5))
+  (segment (start 117.1 66.125) (end 110.625 72.6) (width 0.3) (layer F.Cu) (net 5))
+  (segment (start 110.625 72.6) (end 106.368002 72.6) (width 0.3) (layer F.Cu) (net 5))
   (segment (start 102.74 72.6) (end 106.368002 72.6) (width 0.3) (layer F.Cu) (net 5))
-  (segment (start 106.368002 72.6) (end 115.1 63.868002) (width 0.3) (layer F.Cu) (net 5))
-  (segment (start 115.1 63.868002) (end 115.1 61.825) (width 0.3) (layer F.Cu) (net 5))
-  (segment (start 115.1 61.825) (end 115.1 60.85) (width 0.3) (layer F.Cu) (net 5))
   (segment (start 83.16 72.67) (end 84.190001 73.700001) (width 0.3) (layer F.Cu) (net 5))
   (segment (start 84.190001 73.700001) (end 101.639999 73.700001) (width 0.3) (layer F.Cu) (net 5))
@@
   (segment (start 98.02 95.29) (end 98.34 94.97) (width 0.3) (layer F.Cu) (net 5))
   (segment (start 98.34 94.97) (end 98.34 94.02) (width 0.3) (layer F.Cu) (net 5))
+  (segment (start 114.5 65.15) (end 114.5 65.625) (width 0.3) (layer F.Cu) (net 9))
+  (segment (start 114.5 65.625) (end 110.195 69.93) (width 0.3) (layer F.Cu) (net 9))
+  (segment (start 110.195 69.93) (end 108.42132 69.93) (width 0.3) (layer F.Cu) (net 9))
+  (segment (start 108.42132 69.93) (end 106.3 69.93) (width 0.3) (layer F.Cu) (net 9))
+  (segment (start 128.4 60.8) (end 126.55 60.8) (width 0.3) (layer F.Cu) (net 9))
+  (segment (start 126.55 60.8) (end 125.7 61.65) (width 0.3) (layer F.Cu) (net 9))
   (segment (start 125.7 63) (end 125.7 61.8) (width 0.3) (layer F.Cu) (net 9))
   (segment (start 125.65 74.3) (end 125.65 73.1) (width 0.3) (layer F.Cu) (net 9))
@@
   (segment (start 73 70) (end 75.67 72.67) (width 0.3) (layer F.Cu) (net 9))
   (segment (start 75.67 72.67) (end 76.05 72.67) (width 0.3) (layer F.Cu) (net 9))
-  (segment (start 117.7 60.85) (end 117.7 60.375) (width 0.3) (layer F.Cu) (net 9))
-  (segment (start 117.7 60.375) (end 118.05001 60.02499) (width 0.3) (layer F.Cu) (net 9))
-  (segment (start 118.05001 60.02499) (end 125.77499 60.02499) (width 0.3) (layer F.Cu) (net 9))
-  (segment (start 125.77499 60.02499) (end 126.55 60.8) (width 0.3) (layer F.Cu) (net 9))
-  (segment (start 128.4 60.8) (end 126.55 60.8) (width 0.3) (layer F.Cu) (net 9))
-  (segment (start 126.55 60.8) (end 125.7 61.65) (width 0.3) (layer F.Cu) (net 9))
   (segment (start 125.7 61.65) (end 125.7 61.8) (width 0.3) (layer F.Cu) (net 9))
   (segment (start 128.15 100.9) (end 126.45 100.9) (width 0.3) (layer B.Cu) (net 9))
@@
   (segment (start 75.8 94.02) (end 75.8 92.75) (width 0.3) (layer F.Cu) (net 9))
   (segment (start 75.8 95.29) (end 75.8 94.02) (width 0.3) (layer F.Cu) (net 9))
-  (segment (start 113.9 60.85) (end 118.9 60.85) (width 0.3) (layer B.Cu) (net 10))
-  (segment (start 112.9 63.55) (end 112.9 61.7) (width 0.3) (layer F.Cu) (net 10))
-  (segment (start 112.9 61.7) (end 113.75 60.85) (width 0.3) (layer F.Cu) (net 10))
-  (segment (start 113.75 60.85) (end 113.9 60.85) (width 0.3) (layer F.Cu) (net 10))
-  (segment (start 119.9 63.55) (end 119.9 61.7) (width 0.3) (layer F.Cu) (net 10))
-  (segment (start 119.9 61.7) (end 119.05 60.85) (width 0.3) (layer F.Cu) (net 10))
-  (segment (start 119.05 60.85) (end 118.9 60.85) (width 0.3) (layer F.Cu) (net 10))
+  (segment (start 119.3 62.45) (end 118.5 62.45) (width 0.3) (layer F.Cu) (net 10))
+  (segment (start 118.5 62.45) (end 112.3 62.45) (width 0.3) (layer F.Cu) (net 10))
+  (segment (start 118.3 65.15) (end 118.45 65.15) (width 0.3) (layer F.Cu) (net 10))
+  (segment (start 118.45 65.15) (end 119.3 64.3) (width 0.3) (layer F.Cu) (net 10))
+  (segment (start 119.3 64.3) (end 119.3 63.525) (width 0.3) (layer F.Cu) (net 10))
+  (segment (start 119.3 63.525) (end 119.3 62.45) (width 0.3) (layer F.Cu) (net 10))
+  (segment (start 112.3 62.45) (end 112.3 64.3) (width 0.3) (layer F.Cu) (net 10))
+  (segment (start 112.3 64.3) (end 113.15 65.15) (width 0.3) (layer F.Cu) (net 10))
+  (segment (start 113.15 65.15) (end 113.3 65.15) (width 0.3) (layer F.Cu) (net 10))
   (segment (start 125.45 98.05) (end 117.65 98.05) (width 0.3) (layer F.Cu) (net 12))
   (segment (start 115.57 95.97) (end 115.57 91.44) (width 0.3) (layer F.Cu) (net 12))
@@
   (segment (start 124.124989 76.092891) (end 124.61788 75.6) (width 0.3) (layer F.Cu) (net 21))
   (segment (start 124.675 75.6) (end 125.65 75.6) (width 0.3) (layer F.Cu) (net 21))
+  (segment (start 112.949999 76.725001) (end 124.725 64.95) (width 0.3) (layer F.Cu) (net 24))
   (segment (start 113.03 86.24) (end 113.03 84.84) (width 0.3) (layer F.Cu) (net 24))
   (segment (start 113.03 84.84) (end 112.949999 84.759999) (width 0.3) (layer F.Cu) (net 24))
   (segment (start 112.949999 84.759999) (end 112.949999 76.725001) (width 0.3) (layer F.Cu) (net 24))
-  (segment (start 112.949999 76.725001) (end 124.725 64.95) (width 0.3) (layer F.Cu) (net 24))
   (segment (start 124.725 64.95) (end 125.7 64.95) (width 0.3) (layer F.Cu) (net 24))
+  (segment (start 126.725001 64.350001) (end 126.725001 67.091739) (width 0.3) (layer F.Cu) (net 25))
   (segment (start 125.7 64.3) (end 126.675 64.3) (width 0.3) (layer F.Cu) (net 25))
   (segment (start 126.675 64.3) (end 126.725001 64.350001) (width 0.3) (layer F.Cu) (net 25))
-  (segment (start 126.725001 64.350001) (end 126.725001 67.091739) (width 0.3) (layer F.Cu) (net 25))
   (segment (start 126.725001 67.091739) (end 116.774999 77.041741) (width 0.3) (layer F.Cu) (net 25))
   (segment (start 116.774999 77.041741) (end 116.774999 79.2) (width 0.3) (layer F.Cu) (net 25))

Commit message: update;
Routing:
- added copper zone on B.Cu, net (none)
- added copper zone on F.Cu, net (none)
Changed lines of the file:
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@@
     (links 59)
     (no_connects 0)
-    (area 70.984999 56.215 133.135 103.275)
+    (area 70 57.815 133.135 104.081088)
     (thickness 1.6)
     (drawings 0)
@@
     (last_trace_width 0.25)
     (trace_clearance 0.2)
-    (zone_clearance 0.508)
+    (zone_clearance 1)
     (zone_45_only no)
     (trace_min 0.2)
@@
     (visible_elements 7FFFFFFF)
     (pcbplotparams
-      (layerselection 0x00030_80000001)
+      (layerselection 0x00000_80000000)
       (usegerberextensions false)
       (excludeedgelayer true)
-      (linewidth 0.100000)
+      (linewidth 2.000000)
       (plotframeref false)
       (viasonmask false)
@@
       (hpglpendiameter 15)
       (hpglpenoverlay 2)
-      (psnegative false)
+      (psnegative true)
       (psa4output false)
       (plotreference true)
@@
       (subtractmaskfromsilk false)
       (outputformat 4)
-      (mirror false)
-      (drillshape 0)
+      (mirror true)
+      (drillshape 2)
       (scaleselection 1)
       (outputdirectory output.d))
@@
   (segment (start 83.42 95.29) (end 83 95.29) (width 0.3) (layer F.Cu) (net 30))
   (segment (start 83.42 95.29) (end 92.63 95.29) (width 0.3) (layer F.Cu) (net 30))
+  (zone (net 0) (net_name "") (layer B.Cu) (hatch edge 0.508)
+    (connect_pads (clearance 1))
+    (min_thickness 1)
+    (fill yes (arc_segments 16) (thermal_gap 1) (thermal_bridge_width 2))
+    (polygon
+      (pts
+        (xy 70 58) (xy 70 104) (xy 132 104) (xy 132 58)
+      )
+    )
+  )
+  (zone (net 0) (net_name "") (layer F.Cu) (hatch edge 0.508)
+    (connect_pads (clearance 1))
+    (min_thickness 1)
+    (fill yes (arc_segments 16) (thermal_gap 1) (thermal_bridge_width 2))
+    (polygon
+      (pts
+        (xy 70 58.081087) (xy 70 104.081087) (xy 132 104.081087) (xy 132 58.081087)
+      )
+    )
+  )
 )

Commit message: update
Parts:
- SW1: footprint Buttons_Switches_SMD:SW_DIP_x4_W7.62mm_Slide_Copal_CHS-B -> Buttons_Switches_SMD:SW_DIP_x4_W8.61mm_Slide_LowProfile
- moved REF** 4.94 mm to (86.4, 81.2)
- moved R1 3.44 mm to (94.2, 90.2)
- moved R3 3.40 mm to (94.2, 95.2)
- moved R4 2.59 mm to (94.2, 97.8)
- moved SW1 0.64 mm to (79.8, 94.0)
- moved R2 0.64 mm to (94.2, 92.6)
Routing:
- net Net-(R4-Pad2): track 45.4 -> 32.7 mm
- net Net-(R3-Pad2): track 13.0 -> 9.17 mm
- net GND: track 162.7 -> 165.4 mm
- net VBUS: track 79.9 -> 78.6 mm
- net Net-(J1-Pad3): track 47.5 -> 48.6 mm
- net Net-(R1-Pad2): track 49.6 -> 48.9 mm
