File: QuadUSBSwitch/QuadUSBSwitch.sch (KiCad schematic (older format))
At the start: 13 parts, among them J1 USB_A, J2 USB_A, J3 USB_OTG, J4 USB_OTG, J5 USB_OTG, J6 USB_OTG, J7 USB_OTG, SW1 SW_DIP_x04, U1 CH440G

Commit message: update
Parts:
- SW1: footprint Buttons_Switches_SMD:SW_DIP_x4_W7.62mm_Slide_Copal_CHS-B -> Buttons_Switches_SMD:SW_DIP_x4_W8.61mm_Slide_LowProfile
Changed lines of the file:
@@
 F 0 "SW1" H 1700 4700 50  0000 C CNN
 F 1 "SW_DIP_x04" H 1700 4100 50  0000 C CNN
-F 2 "Buttons_Switches_SMD:SW_DIP_x4_W7.62mm_Slide_Copal_CHS-B" H 1700 4350 50  0001 C CNN
+F 2 "Buttons_Switches_SMD:SW_DIP_x4_W8.61mm_Slide_LowProfile" H 1700 4350 50  0001 C CNN
 F 3 "" H 1700 4350 50  0001 C CNN
 	1    1700 4350
@@
 Connection ~ 5550 5050
 Wire Wire Line
-	2000 4450 4400 4450
+	4400 4450 2000 4450
 Wire Wire Line
 	2000 3100 2000 4150
